File: STM32L152CCx_HARDWARE/REV_1.1/STM32L152Cxx_Module.sch (KiCad schematic (older format))
At the start: 44 parts, among them J1 USB_MINI_B_SMD, P1 CONN_1x20, P2 CONN_1x20, P3 CONN_1x4, P4 Header_2x1, P5 CONN_1x3, SW1 PUSHBUTTON_SPST_3X4MM, U1 LM1117_SOT223, U2 STM32L152Cxx, U3 24FCxx_/MS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

Commit message: Revision 1.1 with open issues corrected & closed
Parts:
- added C14: 33uF, Kicad:CAPACITOR_TANTALUM_B, symbol 47uF_Pol
- added D7: SMLJ33ABCT, Kicad:SOD123F, symbol SMLJ33ABCT
- added D8: BAT54C, Kicad:SOT23-3, symbol BAT54C
- added F3: FUSE_PTC_.5A_33V, Kicad:P1210, symbol FUSE_PTC_.5A_33V
- C1, C2: value 47uF -> 33uF; footprint Kicad:CAPACITOR_TANTALUM_C -> Kicad:CAPACITOR_TANTALUM_B
- D1: footprint Kicad:MINI_SMA -> Kicad:SOD323F
- D3: footprint Kicad:MINI_SMA -> Kicad:SOD123F
Connections:
- net labels added: +3.3V_DIR, +3.3V_EXT, NC, VBAT_EXT
- net labels removed: +3.3V_INT
- wire segments 212 -> 220
Other:
- note added: "1.1\n"
- note added: "NOTES REV 1.0:\n1. +3.3V OUT (P1-2, P2-2) ONLY AVAILABLE \n WHEN POWERED THROUGH +5V LINES\n2. USB PORT BY DEFAULT IS UNPOWERED\n3. BOARD CANNOT BE POWERED THROUGH USB PORT\n4. I2C PULLUPS ON I2C1 BUS 1 ONLY TO SUPPORT EEPROM \n USER MUST PROVIDE PULL-UPS FOR OTHER I2C BUSSES\n5. USE OF I2C INTERNAL PULL-UPS ONLY NOT ADVISED\n6. PB2 USED FOR ONBOARD USER LED. MAY BE \n DISABLED BY REMOVING R7\n\n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"
- note removed: "1.0"
- note removed: "NOTES REV 1.0:\n1. +3.3V OUT (P1-2, P2-2) ONLY AVAILABLE \n WHEN POWERED THROUGH +5V LINES\n2. USB PORT BY DEFAULT IS UNPOWERED\n3. BOARD CANNOT BE POWERED THROUGH USB PORT\n4. I2C PULLUPS ON I2C1 BUS 1 ONLY TO SUPPORT EEPROM \n USER MUST PROVIDE PULL-UPS FOR OTHER I2C BUSSES\n5. USE OF I2C INTERNAL PULL-UPS ONLY NOT ADVISED\n6. PB2 USED FOR ONBOARD USER LED. MAY BE \n DISABLED BY REMOVING R7"
- moved on the sheet: P5, R10, R11
Changed lines of the file:
@@
 Text Label 2325 6950 0    60   ~ 0
 PA10
-Text Label 2325 6850 0    60   ~ 0
+Text Label 2325 6650 0    60   ~ 0
 PA15
-Text Label 2325 6750 0    60   ~ 0
+Text Label 2325 6550 0    60   ~ 0
 PB3
-Text Label 2325 6650 0    60   ~ 0
+Text Label 2325 6450 0    60   ~ 0
 PB4
-Text Label 2325 6550 0    60   ~ 0
+Text Label 2325 6350 0    60   ~ 0
 PB5
-Text Label 2325 6450 0    60   ~ 0
+Text Label 2325 6250 0    60   ~ 0
 PB6
-Text Label 2325 6350 0    60   ~ 0
+Text Label 2325 6150 0    60   ~ 0
 PB7
-Text Label 2325 6250 0    60   ~ 0
+Text Label 2325 6050 0    60   ~ 0
 PB8
-Text Label 2325 6150 0    60   ~ 0
+Text Label 2325 5950 0    60   ~ 0
 PB9
 $Comp
@@
 $EndComp
 Text Label 950  6050 0    60   ~ 0
-VBAT
+VBAT_EXT
 Wire Wire Line
 	1550 2725 1100 2725
@@
 +5V
 Text Label 2325 5750 0    60   ~ 0
-+5V
-Text Label 950  5850 0    60   ~ 0
-+3.3V_OUT
-Text Label 2325 5850 0    60   ~ 0
 +3.3V_OUT
 Wire Wire Line
@@
 Text Label 2325 7650 0    60   ~ 0
 GND
-Text Label 950  5950 0    60   ~ 0
-+3.3V_IN
-Text Label 2325 5950 0    60   ~ 0
+Text Label 2325 5850 0    60   ~ 0
 +3.3V_IN
 $Comp
 L CONN_1x3 P5
 U 1 1 5ADFC3BE
-P 8625 6300
-F 0 "P5" H 8675 6350 60  0000 C CNN
-F 1 "CONN_1x3" H 8850 5950 60  0000 C CNN
-F 2 "Kicad:HEADER_1X3_2MM" H 8625 6300 60  0001 C CNN
-F 3 "" H 8625 6300 60  0000 C CNN
-	1    8625 6300
+P 7775 6300
+F 0 "P5" H 7825 6350 60  0000 C CNN
+F 1 "CONN_1x3" H 8000 5950 60  0000 C CNN
+F 2 "Kicad:HEADER_1X3_2MM" H 7775 6300 60  0001 C CNN
+F 3 "" H 7775 6300 60  0000 C CNN
+	1    7775 6300
 	1    0    0    -1
 $EndComp
@@
 F 0 "D3" H 9250 3175 50  0000 C CNN
 F 1 "SMLJ33ABCT" H 9250 2975 50  0001 C CNN
-F 2 "Kicad:MINI_SMA" H 9250 3075 50  0001 C CNN
+F 2 "Kicad:SOD123F" H 9250 3075 50  0001 C CNN
 F 3 "" H 9250 3075 50  0000 C CNN
 	1    9250 3075
@@
 F 0 "D1" H 7250 3225 50  0000 C CNN
 F 1 "SMLJ33ABCT" H 7250 3025 50  0001 C CNN
-F 2 "Kicad:MINI_SMA" H 7250 3125 50  0001 C CNN
+F 2 "Kicad:SOD323F" H 7250 3125 50  0001 C CNN
 F 3 "" H 7250 3125 50  0000 C CNN
 	1    7250 3125
@@
 P 7050 3025
 F 0 "C1" H 7300 3100 60  0000 C CNN
-F 1 "47uF" H 7175 2925 60  0000 C CNN
-F 2 "Kicad:CAPACITOR_TANTALUM_C" H 7050 3025 60  0001 C CNN
+F 1 "33uF" H 7175 2925 60  0000 C CNN
+F 2 "Kicad:CAPACITOR_TANTALUM_B" H 7050 3025 60  0001 C CNN
 F 3 "" H 7050 3025 60  0000 C CNN
 	1    7050 3025
@@
 P 8675 2975
 F 0 "C2" H 8925 3050 60  0000 C CNN
-F 1 "47uF" H 8800 2875 60  0000 C CNN
-F 2 "Kicad:CAPACITOR_TANTALUM_C" H 8675 2975 60  0001 C CNN
+F 1 "33uF" H 8800 2875 60  0000 C CNN
+F 2 "Kicad:CAPACITOR_TANTALUM_B" H 8675 2975 60  0001 C CNN
 F 3 "" H 8675 2975 60  0000 C CNN
 	1    8675 2975
@@
 +3.3V_OUT
 Wire Wire Line
-	8425 6550 7975 6550
-Wire Wire Line
-	8425 6450 7975 6450
-Wire Wire Line
-	8425 6350 7975 6350
-Text Label 7975 6450 0    60   ~ 0
+	5700 6550 7575 6550
+Wire Wire Line
+	7575 6450 7125 6450
+Wire Wire Line
+	7575 6350 7125 6350
+Text Label 7125 6450 0    60   ~ 0
 +3.3V
-Text Label 7975 6350 0    60   ~ 0
-+3.3V_INT
-Text Label 7975 6550 0    60   ~ 0
-+3.3V_IN
 $Comp
 L 0.10uF C8
@@
 	5475 900  5475 950
 Wire Wire Line
-	4075 900  5475 900
+	4075 900  5800 900
 Wire Wire Line
 	4075 900  4075 950
@@
 	4075 1200 4075 1250
 Wire Wire Line
-	4075 1250 5475 1250
+	4075 1250 5800 1250
 Wire Wire Line
 	5475 1250 5475 1200
@@
 	2775 5950 2325 5950
 Text Label 8550 2950 0    60   ~ 0
-+3.3V_INT
++3.3V_EXT
 $Comp
 L PUSHBUTTON_SPST_3X4MM SW1
@@
 May 23rd, 2018
 Text Notes 10000 7875 0    60   ~ 0
-1.0
+1.1\n
 Text Notes 6500 6075 0    60   ~ 0
 +3.3V POWER SOURCE SELECTION\n1-2 - SOURCED FROM +5V  TO +12V  IN THROUGH LDO REGULATOR (P1-1, P2-1\n2-3 - SOURCED FROM EXTERNAL +3.3 REGULATED SOURCE (P1-3, P2-3)
@@
 Text Notes 1475 2500 0    60   ~ 0
 STM32L152CCx PROCESSOR
-Text Notes 625  1525 0    60   ~ 0
-NOTES REV 1.0:\n1. +3.3V OUT (P1-2, P2-2) ONLY AVAILABLE \n    WHEN POWERED THROUGH +5V LINES\n2. USB PORT BY DEFAULT IS UNPOWERED\n3. BOARD CANNOT BE POWERED THROUGH USB PORT\n4. I2C PULLUPS ON I2C1 BUS 1 ONLY TO SUPPORT EEPROM \n    USER MUST PROVIDE PULL-UPS FOR OTHER I2C BUSSES\n5. USE OF I2C INTERNAL PULL-UPS ONLY NOT ADVISED\n6. PB2 USED FOR ONBOARD USER LED. MAY BE \n    DISABLED BY REMOVING R7
+Text Notes 575  2225 0    60   ~ 0
+NOTES REV 1.0:\n1. +3.3V OUT (P1-2, P2-2) ONLY AVAILABLE \n    WHEN POWERED THROUGH +5V LINES\n2. USB PORT BY DEFAULT IS UNPOWERED\n3. BOARD CANNOT BE POWERED THROUGH USB PORT\n4. I2C PULLUPS ON I2C1 BUS 1 ONLY TO SUPPORT EEPROM \n    USER MUST PROVIDE PULL-UPS FOR OTHER I2C BUSSES\n5. USE OF I2C INTERNAL PULL-UPS ONLY NOT ADVISED\n6. PB2 USED FOR ONBOARD USER LED. MAY BE \n    DISABLED BY REMOVING R7\n\nNOTES REV 1.0 -> 1.1\n1. REVISED BOARD PINOUTS\n2. BROUGHT OUT USB PINS TO HEADERS\n3. REVISED +3.3V CORE SWITCHING\n4. ADDED DIODE BLOCEKD POWER TO VBAT IF\n    EXT VBAT NOT PRESENT
 $Comp
 L 3.30kΩ R10
 U 1 1 5B078E46
-P 4725 6175
-F 0 "R10" H 4800 6275 60  0000 C CNN
-F 1 "3.30kΩ" H 5075 6275 60  0000 C CNN
-F 2 "Kicad:P0603" H 4725 6175 60  0001 C CNN
-F 3 "" H 4915 6245 60  0000 C CNN
-	1    4725 6175
+P 4375 6025
+F 0 "R10" H 4450 6125 60  0000 C CNN
+F 1 "3.30kΩ" H 4725 6125 60  0000 C CNN
+F 2 "Kicad:P0603" H 4375 6025 60  0001 C CNN
+F 3 "" H 4565 6095 60  0000 C CNN
+	1    4375 6025
 	1    0    0    -1
 $EndComp
@@
 L 3.30kΩ R11
 U 1 1 5B078F2F
-P 4725 6425
-F 0 "R11" H 4800 6500 60  0000 C CNN
-F 1 "3.30kΩ" H 5075 6500 60  0000 C CNN
-F 2 "Kicad:P0603" H 4725 6425 60  0001 C CNN
-F 3 "" H 4915 6495 60  0000 C CNN
-	1    4725 6425
+P 4375 6275
+F 0 "R11" H 4450 6350 60  0000 C CNN
+F 1 "3.30kΩ" H 4725 6350 60  0000 C CNN
+F 2 "Kicad:P0603" H 4375 6275 60  0001 C CNN
+F 3 "" H 4565 6345 60  0000 C CNN
+	1    4375 6275
 	1    0    0    -1
 $EndComp
@@
 L +3.3V #PWR032
 U 1 1 5B0791F9
-P 5300 6025
-F 0 "#PWR032" H 5300 5875 50  0001 C CNN
-F 1 "+3.3V" H 5300 6165 50  0000 C CNN
-F 2 "" H 5300 6025 50  0000 C CNN
-F 3 "" H 5300 6025 50  0000 C CNN
-	1    5300 6025
-	1    0    0    -1
-$EndComp
-Wire Wire Line
-	5300 6025 5300 6425
-Wire Wire Line
-	5300 6425 5125 6425
-Wire Wire Line
-	5125 6175 5300 6175
-Connection ~ 5300 6175
-Wire Wire Line
-	4725 6175 4325 6175
-Wire Wire Line
-	4725 6425 4325 6425
-Text Label 4325 6175 0    60   ~ 0
+P 4950 5875
+F 0 "#PWR032" H 4950 5725 50  0001 C CNN
+F 1 "+3.3V" H 4950 6015 50  0000 C CNN
+F 2 "" H 4950 5875 50  0000 C CNN
+F 3 "" H 4950 5875 50  0000 C CNN
+	1    4950 5875
+	1    0    0    -1
+$EndComp
+Wire Wire Line
+	4950 5875 4950 6275
+Wire Wire Line
+	4950 6275 4775 6275
+Wire Wire Line
+	4775 6025 4950 6025
+Connection ~ 4950 6025
+Wire Wire Line
+	4375 6025 3975 6025
+Wire Wire Line
+	4375 6275 3975 6275
+Text Label 3975 6025 0    60   ~ 0
 PB10
-Text Label 4325 6425 0    60   ~ 0
+Text Label 3975 6275 0    60   ~ 0
 PB11
-Text Notes 4525 5675 0    60   ~ 0
+Text Notes 4175 5525 0    60   ~ 0
 I2C1 PULL-UPS
+Text Label 7125 6350 0    60   ~ 0
++3.3V_EXT
+$Comp
+L FUSE_PTC_.5A_33V F3
+U 1 1 5B173B50
+P 5500 6550
+F 0 "F3" H 5350 6450 60  0000 C CNN
+F 1 "FUSE_PTC_.5A_33V" H 5600 6700 60  0001 C CNN
+F 2 "Kicad:P1210" H 5500 6550 60  0001 C CNN
+F 3 "" H 5500 6550 60  0000 C CNN
+	1    5500 6550
+	1    0    0    -1
+$EndComp
+$Comp
+L SMLJ33ABCT D7
+U 1 1 5B173CCE
+P 5775 6700
+F 0 "D7" H 5775 6800 50  0000 C CNN
+F 1 "SMLJ33ABCT" H 5775 6600 50  0001 C CNN
+F 2 "Kicad:SOD123F" H 5775 6700 50  0001 C CNN
+F 3 "" H 5775 6700 50  0000 C CNN
+	1    5775 6700
+	0    1    1    0
+$EndComp
+$Comp
+L GND #PWR033
+U 1 1 5B173EAA
+P 5775 6850
+F 0 "#PWR033" H 5775 6600 50  0001 C CNN
+F 1 "GND" H 5775 6700 50  0000 C CNN
+F 2 "" H 5775 6850 50  0000 C CNN
+F 3 "" H 5775 6850 50  0000 C CNN
+	1    5775 6850
+	1    0    0    -1
+$EndComp
+Wire Wire Line
+	5300 6550 4800 6550
+Wire Wire Line
+	5775 6600 5775 6550
+Connection ~ 5775 6550
+Wire Wire Line
+	5775 6850 5775 6800
+Text Label 4800 6550 0    60   ~ 0
++3.3V_IN
+Text Label 7125 6550 0    60   ~ 0
++3.3V_DIR
+$Comp
+L 47uF_Pol C14
+U 1 1 5B1759BE
+P 5800 950
+F 0 "C14" H 6050 1025 60  0000 C CNN
+F 1 "33uF" H 5925 850 60  0000 C CNN
+F 2 "Kicad:CAPACITOR_TANTALUM_B" H 5800 950 60  0001 C CNN
+F 3 "" H 5800 950 60  0000 C CNN
+	1    5800 950
+	0    1    1    0
+$EndComp
+Wire Wire Line
+	5800 900  5800 950
+Connection ~ 5475 900
+Wire Wire Line
+	5800 1250 5800 1200
+Connection ~ 5475 1250
+Text Label 950  5950 0    60   ~ 0
+NC
+$Comp
+L BAT54C D8
+U 1 1 5B198271
+P 4550 7300
+F 0 "D8" H 4600 7425 60  0000 C CNN
+F 1 "BAT54C" H 4700 6975 60  0000 C CNN
+F 2 "Kicad:SOT23-3" H 4550 7300 60  0001 C CNN
+F 3 "" H 4550 7300 60  0001 C CNN
+	1    4550 7300
+	1    0    0    -1
+$EndComp
+Wire Wire Line
+	4750 7400 5125 7400
+Wire Wire Line
+	4450 7300 4075 7300
+Wire Wire Line
+	4450 7500 4075 7500
+Text Label 4900 7400 0    60   ~ 0
+VBAT
+Text Label 4075 7500 0    60   ~ 0
++3.3V
+Text Label 4075 7300 0    60   ~ 0
+VBAT_EXT
+Text Label 2325 6750 0    60   ~ 0
+USB_DP
+Text Label 2325 6850 0    60   ~ 0
+USB_DM
+Text Label 950  5850 0    60   ~ 0
+NC
 $EndSCHEMATC
