File: STM32L152CCx_HARDWARE/REV_1.1/STM32L152Cxx_Module.kicad_pcb (KiCad board)
At the start: 4 copper layers, 50.8 x 20.3 mm, 52 parts, among them J1 USB_MINI_B_SMD, P1 CONN_1x20, P2 CONN_1x20, P3 CONN_1x4, P4 Header_2x1, P5 CONN_1x3, SW1 PUSHBUTTON_SPST_3X4MM, U1 LM1117_SOT223, U2 STM32L152Cxx, U3 24FCxx_/MS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

Commit message: Update 7/4/2018
Other:
- board text added: "C G D"
- board text added: "STM32L152CC REV 1.1"
- board text removed: "STM32L152CC REV1"
- board text removed: "V C G D"
Changed lines of the file:
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@@
       (drillshape 0)
       (scaleselection 1)
-      (outputdirectory CAM/))
+      (outputdirectory STM32L152Cxx_CAM/))
   )
   (net 0 "")
@@
     (tags CHIP)
     (attr smd)
-    (fp_text reference F2 (at -2.8 0.15 90) (layer B.SilkS)
+    (fp_text reference F2 (at -2.81 -1.17 180) (layer B.SilkS)
       (effects (font (size 0.75 0.75) (thickness 0.1)) (justify mirror))
     )
@@
     (tags CHIP)
     (attr smd)
-    (fp_text reference F1 (at 3.175 -0.127) (layer B.SilkS)
+    (fp_text reference F1 (at 2.98 0.86) (layer B.SilkS)
       (effects (font (size 0.75 0.75) (thickness 0.1)) (justify mirror))
     )
@@
   (module Kicad:SWITCH_SPST_3X4MM (layer F.Cu)
     (at 99.695 128.905 180)
-    (fp_text reference SW1 (at -1.605 -2.645 180) (layer F.SilkS)
+    (fp_text reference SW1 (at 4.465 -0.005 180) (layer F.SilkS)
       (effects (font (size 0.75 0.75) (thickness 0.1)))
     )
@@
   (module Kicad:CAPACITOR_TANTALUM_B (layer B.Cu)
     (at 60.95 130.15 180)
-    (fp_text reference C14 (at -0.127 2.413 180) (layer B.SilkS)
+    (fp_text reference C14 (at 1.72 2.64 180) (layer B.SilkS)
       (effects (font (size 0.7 0.7) (thickness 0.1)) (justify mirror))
     )
@@
     (tags CHIP)
     (attr smd)
-    (fp_text reference F3 (at 2.75 0 270) (layer B.SilkS)
+    (fp_text reference F3 (at 2.86 0.12 360) (layer B.SilkS)
       (effects (font (size 0.65 0.65) (thickness 0.0975)) (justify mirror))
     )
@@
   (module Kicad:FIDUCIAL_BOTTOM (layer F.Cu)
     (at 61.38 127.01)
-    (fp_text reference REF** (at 0.7112 -2.0828) (layer F.SilkS)
+    (fp_text reference REF** (at -0.9 -0.55) (layer F.SilkS) hide
       (effects (font (size 0.7 0.7) (thickness 0.1)))
     )
@@
     (effects (font (size 2 2) (thickness 0.3)) (justify left))
   )
-  (gr_text "V\n\nC\n\nG\n\nD" (at 65 120 90) (layer F.SilkS)
+  (gr_text "C\n\nG\n\nD" (at 66.33 120.01 90) (layer F.SilkS)
     (effects (font (size 0.8 0.8) (thickness 0.15)))
   )
-  (gr_text "STM32L152CC REV1" (at 80.45 131.3) (layer F.SilkS)
+  (gr_text "STM32L152CC REV 1.1" (at 83.33 131.485) (layer F.SilkS)
     (effects (font (size 1 1) (thickness 0.15)))
   )
